File: Noname.kicad_pcb (KiCad board)
At the start: 2 copper layers, 234.4 x 87.4 mm, 77 parts, among them SW1 SW_PUSH, SW10 SW_PUSH, SW11 SW_PUSH, SW12 SW_PUSH, SW13 SW_PUSH, SW14 SW_PUSH, SW15 SW_PUSH, SW16 SW_PUSH, SW17 SW_PUSH, SW18 SW_PUSH, SW19 SW_PUSH, SW2 SW_PUSH, SW20 SW_PUSH, SW21 SW_PUSH, SW22 SW_PUSH, SW23 SW_PUSH, SW24 SW_PUSH, SW25 SW_PUSH, SW26 SW_PUSH, SW27 SW_PUSH, SW28 SW_PUSH, SW29 SW_PUSH, SW3 SW_PUSH, SW30 SW_PUSH, SW31 SW_PUSH, SW32 SW_PUSH, SW33 SW_PUSH, SW34 SW_PUSH, SW35 SW_PUSH, SW36 SW_PUSH, SW37 SW_PUSH, SW4 SW_PUSH, SW5 SW_PUSH, SW6 SW_PUSH, SW7 SW_PUSH, SW8 SW_PUSH, SW9 SW_PUSH, U1 ProMicro_r

Commit message: Update v1.3
Parts:
- removed OL1: OLED, KBD:OLED_v2
- added D39: WS2812B, KBD:LED_WS2812B-PLCC4, B.Cu at (250.6, 120.5)
- added D40: WS2812B, KBD:LED_WS2812B-PLCC4, B.Cu at (205.0, 138.6)
- added D41: WS2812B, KBD:LED_WS2812B-PLCC4, B.Cu at (145.6, 148.0)
- added D42: WS2812B, KBD:LED_WS2812B-PLCC4, B.Cu at (145.6, 114.0)
- added D43: WS2812B, KBD:LED_WS2812B-PLCC4, B.Cu at (86.3, 138.6)
- added D44: WS2812B, KBD:LED_WS2812B-PLCC4, B.Cu at (40.7, 120.5)
- added D45: WS2812B, KBD:LED_WS2812B-PLCC4, B.Cu at (45.3, 82.7)
- added D46: WS2812B, KBD:LED_WS2812B-PLCC4, B.Cu at (118.7, 66.7)
- D1, D10, D11, D12, D13, D14, D15, D16, D17, D18, D19, D2, D20, D21, D22, D23, D24, D25, D26, D27, D28, D29, D3, D30, D31, D32, D33, D34, D35, D36, D4, D5, D6, D7, D8, D9: value D -> 1N4148W
- D37, D38: footprint LED_SMD:LED_WS2812B_PLCC4_5.0x5.0mm_P3.2mm -> KBD:LED_WS2812B-PLCC4
- SW1, SW10, SW11, SW12, SW13, SW14, SW15, SW16, SW17, SW18, SW19, SW2, SW20, SW21, SW22, SW23, SW24, SW25, SW26, SW27, SW28, SW29, SW3, SW30, SW31, SW32, SW35, SW36, SW4, SW5, SW6, SW7, SW8, SW9: footprint KBD:CherryMX_1u -> KBD:CherryMX_Hotswap
- SW33, SW34: footprint KBD:CherryMX_1u -> KBD:CherryMX_Hotswap_1.5u
- U1: value ProMicro_r -> ProMicro; moved to F.Cu
- moved D38 105.6 mm to (246.0, 82.7), turned to -173 degrees
- moved D37 53.7 mm to (172.6, 66.7), turned to -173 degrees
- moved D35 34.4 mm to (175.3, 129.3), turned to -90 degrees
- moved D36 33.6 mm to (194.3, 124.3), turned to -90 degrees
- moved D34 30.1 mm to (160.2, 129.3), turned to -90 degrees
- moved SW34 29.8 mm to (162.7, 144.4), turned to -53 degrees
- moved SW33 25.9 mm to (128.6, 144.4), turned to 53 degrees
- moved SW35 24.9 mm to (184.3, 138.0), turned to 22 degrees
- moved SW36 21.5 mm to (205.0, 132.6)
- moved SW32 21.0 mm to (107.0, 138.0), turned to -22 degrees
- moved D4 20.0 mm to (110.1, 82.4)
- moved D14 20.0 mm to (107.8, 101.4)
- moved D24 20.0 mm to (105.4, 120.3)
- moved D27 18.2 mm to (201.0, 117.9)
- moved D7 18.2 mm to (196.4, 80.0)
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Connections:
- D1 pad 1: R0 -> ROW01
- D10 pad 1: R0 -> ROW01
- D11 pad 1: R1 -> ROW02
- D12 pad 1: R1 -> ROW02
- D13 pad 1: R1 -> ROW02
- D14 pad 1: R1 -> ROW02
- D15 pad 1: R1 -> ROW02
- D16 pad 1: R1 -> ROW02
- D17 pad 1: R1 -> ROW02
- D18 pad 1: R1 -> ROW02
- D19 pad 1: R1 -> ROW02
- D2 pad 1: R0 -> ROW01
- D20 pad 1: R1 -> ROW02
- D21 pad 1: R2 -> ROW03
- D22 pad 1: R2 -> ROW03
- D23 pad 1: R2 -> ROW03
- D24 pad 1: R2 -> ROW03
- D25 pad 1: R2 -> ROW03
- D26 pad 1: R2 -> ROW03
- D27 pad 1: R2 -> ROW03
- D28 pad 1: R2 -> ROW03
- D29 pad 1: R2 -> ROW03
- D3 pad 1: R0 -> ROW01
- D30 pad 1: R2 -> ROW03
- D31 pad 1: R3 -> ROW04
- D32 pad 1: R3 -> ROW04
- D33 pad 1: R3 -> ROW04
- D34 pad 1: R3 -> ROW04
- D35 pad 1: R3 -> ROW04
- D36 pad 1: R3 -> ROW04
- D38 pad 2: (no net) -> Net-(D38-Pad2)
- D4 pad 1: R0 -> ROW01
- D5 pad 1: R0 -> ROW01
- D6 pad 1: R0 -> ROW01
- D7 pad 1: R0 -> ROW01
- D8 pad 1: R0 -> ROW01
- D9 pad 1: R0 -> ROW01
- SW1 pad 1: C0 -> COL01
- SW10 pad 1: C9 -> COL10
- SW11 pad 1: C0 -> COL01
- SW12 pad 1: C1 -> COL02
- SW13 pad 1: C2 -> COL03
- SW14 pad 1: C3 -> COL04
- SW15 pad 1: C4 -> COL05
- SW16 pad 1: C5 -> COL06
- SW17 pad 1: C6 -> COL07
- SW18 pad 1: C7 -> COL08
- SW19 pad 1: C8 -> COL09
- SW2 pad 1: C1 -> COL02
- SW20 pad 1: C9 -> COL10
- SW21 pad 1: C0 -> COL01
- SW22 pad 1: C1 -> COL02
- SW23 pad 1: C2 -> COL03
- SW24 pad 1: C3 -> COL04
- SW25 pad 1: C4 -> COL05
- SW26 pad 1: C5 -> COL06
- SW27 pad 1: C6 -> COL07
- SW28 pad 1: C7 -> COL08
- SW29 pad 1: C8 -> COL09
- SW3 pad 1: C2 -> COL03
- SW30 pad 1: C9 -> COL10
- SW31 pad 1: C2 -> COL03
- SW32 pad 1: C3 -> COL04
- SW33 pad 1: C4 -> COL05
- SW34 pad 1: C5 -> COL06
- SW35 pad 1: C6 -> COL07
- SW36 pad 1: C7 -> COL08
- SW37 pad 1: GND -> RST
- SW37 pad 2: RS -> GND
- SW4 pad 1: C3 -> COL04
- SW5 pad 1: C4 -> COL05
- SW6 pad 1: C5 -> COL06
- SW7 pad 1: C6 -> COL07
- SW8 pad 1: C7 -> COL08
- SW9 pad 1: C8 -> COL09
- U1 pad 1: R0 -> unconnected-(U1-Pad1)
- U1 pad 10: C2 -> COL08
- U1 pad 11: C1 -> COL07
- U1 pad 12: C0 -> COL06
- U1 pad 13: C9 -> COL05
- U1 pad 14: C8 -> COL04
- U1 pad 15: C7 -> COL03
- U1 pad 16: C6 -> COL02
- U1 pad 17: C5 -> COL01
- U1 pad 18: LED -> unconnected-(U1-Pad18)
- U1 pad 19: R3 -> ROW02
- U1 pad 2: R1 -> unconnected-(U1-Pad2)
- U1 pad 20: R2 -> ROW01
- U1 pad 22: RS -> RST
- U1 pad 24: (no net) -> unconnected-(U1-Pad24)
- U1 pad 5: SDA -> ROW03
- U1 pad 6: SCL -> ROW04
- U1 pad 7: (no net) -> LED
- U1 pad 8: C4 -> COL10
- U1 pad 9: C3 -> COL09
Routing:
- net VCC: track 70.7 -> 622.5 mm, vias 0 -> 11
- net R1: track 282.2 -> 0.00 mm
- net R2: track 280.4 -> 0.00 mm, vias 2 -> 0
- net R0: track 277.9 -> 0.00 mm
- net ROW03: track 0.00 -> 275.7 mm, vias 0 -> 1
- net ROW02: track 0.00 -> 249.3 mm, vias 0 -> 3
- net ROW01: track 0.00 -> 233.0 mm, vias 0 -> 3
- net R3: track 201.0 -> 0.00 mm, vias 2 -> 0
- net C0: track 164.4 -> 0.00 mm, vias 11 -> 0
- net COL01: track 0.00 -> 157.5 mm
- net C2: track 156.2 -> 0.00 mm, vias 8 -> 0
- net COL03: track 0.00 -> 155.2 mm, vias 0 -> 6
- net ROW04: track 0.00 -> 151.7 mm, vias 0 -> 1
- net COL10: track 0.00 -> 149.2 mm, vias 0 -> 8
- net C9: track 147.7 -> 0.00 mm, vias 11 -> 0
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Other:
- board size 234.4 x 87.4 mm -> 231 x 104.9 mm
- board text removed: "Noname by TUS - rev1.0"
